Commit message: Now i can visualize the robot!

File: unitree_description/a1_description/urdf/a1.urdf (robot description, URDF)
Before this commit: robot a1_description, 23 links, 22 joints
Links:
- link FL_calf: geometry collision box size=0.2 0.016 0.016; visual mesh filename=file://$(find a1_description)/meshes/calf.dae scale=1 1 1
- link FL_hip: geometry collision cylinder length=0.04 radius=0.046; visual mesh filename=file://$(find a1_description)/meshes/hip.dae scale=1 1 1
- link FL_thigh: geometry collision box size=0.2 0.0245 0.034; visual mesh filename=file://$(find a1_description)/meshes/thigh.dae scale=1 1 1
- link FR_calf: geometry collision box size=0.2 0.016 0.016; visual mesh filename=file://$(find a1_description)/meshes/calf.dae scale=1 1 1
- link FR_hip: geometry collision cylinder length=0.04 radius=0.046; visual mesh filename=file://$(find a1_description)/meshes/hip.dae scale=1 1 1
- link FR_thigh: geometry collision box size=0.2 0.0245 0.034; visual mesh filename=file://$(find a1_description)/meshes/thigh_mirror.dae scale=1 1 1
- link RL_calf: geometry collision box size=0.2 0.016 0.016; visual mesh filename=file://$(find a1_description)/meshes/calf.dae scale=1 1 1
- link RL_hip: geometry collision cylinder length=0.04 radius=0.046; visual mesh filename=file://$(find a1_description)/meshes/hip.dae scale=1 1 1
- link RL_thigh: geometry collision box size=0.2 0.0245 0.034; visual mesh filename=file://$(find a1_description)/meshes/thigh.dae scale=1 1 1
- link RR_calf: geometry collision box size=0.2 0.016 0.016; visual mesh filename=file://$(find a1_description)/meshes/calf.dae scale=1 1 1
- link RR_hip: geometry collision cylinder length=0.04 radius=0.046; visual mesh filename=file://$(find a1_description)/meshes/hip.dae scale=1 1 1
- link RR_thigh: geometry collision box size=0.2 0.0245 0.034; visual mesh filename=file://$(find a1_description)/meshes/thigh_mirror.dae scale=1 1 1
- link trunk: geometry collision box size=0.267 0.194 0.114; visual mesh filename=file://$(find a1_description)/meshes/trunk.dae scale=1 1 1

File: unitree_description/a1_description/xacro/const.xacro (robot description, xacro)
@@ -4,4 +4,7 @@
     <xacro:property name="PI" value="3.1415926535897931"/>
     <xacro:property name="stick_mass" value="0.00001"/>
+    <!-- Mesh scale correction: meshes are authored in millimeters but interpreted as meters -->
+    <!-- Apply 0.001 scale factor to convert from mm to m -->
+    <xacro:property name="mesh_scale" value="1 1 1"/>
     <!-- simplified collision value -->
     <xacro:property name="trunk_width" value="0.194"/>

File: unitree_description/a1_description/xacro/leg.xacro (robot description, xacro)
@@ -31,5 +31,5 @@
                 </xacro:if>
                 <geometry>
-                    <mesh filename="$(find a1_description)/meshes/hip.dae" scale="1 1 1"/>
+                    <mesh filename="package://a1_description/meshes/hip.dae" scale="${mesh_scale}"/>
                 </geometry>
                 <material name="orange"/>
@@ -77,8 +77,8 @@
                 <geometry>
                     <xacro:if value="${mirror_dae == True}">
-                        <mesh filename="$(find a1_description)/meshes/thigh.dae" scale="1 1 1"/>
+                        <mesh filename="package://a1_description/meshes/thigh.dae" scale="${mesh_scale}"/>
                     </xacro:if>
                     <xacro:if value="${mirror_dae == False}">
-                        <mesh filename="$(find a1_description)/meshes/thigh_mirror.dae" scale="1 1 1"/>
+                        <mesh filename="package://a1_description/meshes/thigh_mirror.dae" scale="${mesh_scale}"/>
                     </xacro:if>
                 </geometry>
@@ -112,5 +112,5 @@
                 <origin rpy="0 0 0" xyz="0 0 0"/>
                 <geometry>
-                    <mesh filename="$(find a1_description)/meshes/calf.dae" scale="1 1 1"/>
+                    <mesh filename="package://a1_description/meshes/calf.dae" scale="${mesh_scale}"/>
                 </geometry>
                 <material name="orange"/>

File: unitree_description/a1_description/xacro/robot.xacro (robot description, xacro)
@@ -39,5 +39,5 @@
             <origin rpy="0 0 0" xyz="0 0 0"/>
             <geometry>
-                <mesh filename="$(find a1_description)/meshes/trunk.dae" scale="1 1 1"/>
+                <mesh filename="package://a1_description/meshes/trunk.dae" scale="${mesh_scale}"/>
             </geometry>
             <material name="orange"/>
