Commit message: Now the robot actually moves. Still very bad movements tho.Add simple simulation and improve control modes.
Introduces a simple robot simulator node for world frame movement and updates launch files for fake simulation. Adds an 'Idling' control mode, improves control mode parsing, and implements basic walking logic in Control mode. Updates hardware plugin registration for Gazebo compatibility, removes foot force sensor dependency for simulation, and refines teleop scripts and setup.

File: unitree_description/a1_description/xacro/robot.xacro (robot description, xacro)
@@ -31,5 +31,5 @@
     </link>
     <joint name="floating_base" type="fixed">
-        <origin rpy="0 0 0" xyz="0 0 0"/>
+        <origin rpy="0 0 0" xyz="0 0 0.25"/>
         <parent link="base"/>
         <child link="trunk"/>
@@ -166,5 +166,8 @@
         <ros2_control name="a1_ros2_control_settings" type="system">
             <hardware>
-                <plugin>unitree_gazebo/UnitreeGazeboSystem</plugin>
+                <!-- <plugin>unitree_gazebo/UnitreeGazeboSystem</plugin> -->
+                <plugin>fake_components/GenericSystem</plugin>
+                <param name="fake_sensor_commands">false</param>
+                <param name="state_following_offset">0.0</param>
                 <!-- <plugin>gazebo_ros2_control/GazeboSystem</plugin> -->
             </hardware>
